File: Pokedex/DexMB.kicad_pcb (KiCad board)
At the start: 2 copper layers, 208.7 x 88.9 mm, 31 parts

Commit message: Completed Files
The Design has been Completed!
Parts:
- removed the ? at (229.2, 123.2) (x2)
- removed the ? at (229.2, 125.1)
- removed Battery: JST_EH_S2B-EH_1x02_P2.50mm_Horizontal, Connector_JST:JST_EH_S2B-EH_1x02_P2.50mm_Horizontal
- removed the REF** at (90.2, 54.7)
- removed the REF** at (220.7, 112.6)
- added 10uF: C_0805_2012Metric, Capacitor_SMD:C_0805_2012Metric, F.Cu at (84.3, 98.0)
- added 10uF: C_0805_2012Metric, Capacitor_SMD:C_0805_2012Metric, F.Cu at (236.1, 120.7)
- added 150: R_0603_1608Metric, Resistor_SMD:R_0603_1608Metric, F.Cu at (88.5, 97.4)
- added 270: R_0603_1608Metric, Resistor_SMD:R_0603_1608Metric, F.Cu at (92.1, 85.6)
- added 270: R_0603_1608Metric, Resistor_SMD:R_0603_1608Metric, F.Cu at (93.4, 84.1)
- added 270: R_0603_1608Metric, Resistor_SMD:R_0603_1608Metric, F.Cu at (89.7, 94.5)
- added 33 nF: C_1206_3216Metric, Capacitor_SMD:C_1206_3216Metric, F.Cu at (86.6, 98.2)
- added ?: , , F.Cu at (88.6, 102.2)
- added ?: , , F.Cu at (86.7, 102.2)
- added BAT: TE_440055-2, Custom GBA Tools:TE_440055-2, B.Cu at (101.4, 108.0)
- added PWM_IN: TE_440055-2, Custom GBA Tools:TE_440055-2, B.Cu at (224.9, 106.1)
- added PWM_OUT: TE_440055-2, Custom GBA Tools:TE_440055-2, B.Cu at (233.8, 106.1)
- added REF**: D_SOD-110, Diode_SMD:D_SOD-110, F.Cu at (107.2, 130.7)
- added REF**: TestPoint_Pad_1.0x1.0mm, TestPoint:TestPoint_Pad_1.0x1.0mm, F.Cu at (107.2, 128.0)
- added REF**: TestPoint_Pad_1.0x1.0mm, TestPoint:TestPoint_Pad_1.0x1.0mm, F.Cu at (223.6, 114.3)
- added REF**: TestPoint_Pad_1.0x1.0mm, TestPoint:TestPoint_Pad_1.0x1.0mm, F.Cu at (107.2, 121.9)
- added REF**: TestPoint_Pad_1.0x1.0mm, TestPoint:TestPoint_Pad_1.0x1.0mm, F.Cu at (225.8, 114.3)
- added REF**: TestPoint_Pad_1.0x1.0mm, TestPoint:TestPoint_Pad_1.0x1.0mm, F.Cu at (107.2, 124.0)
- added REF**: TestPoint_Pad_1.0x1.0mm, TestPoint:TestPoint_Pad_1.0x1.0mm, B.Cu at (107.2, 128.0)
- added REF**: TestPoint_Pad_1.0x1.0mm, TestPoint:TestPoint_Pad_1.0x1.0mm, B.Cu at (219.3, 114.3)
- added REF**: TestPoint_Pad_1.0x1.0mm, TestPoint:TestPoint_Pad_1.0x1.0mm, F.Cu at (219.6, 99.1)
- added REF**: SW_E-Switch_EG1224_SPDT_Angled, Button_Switch_THT:SW_E-Switch_EG1224_SPDT_Angled, B.Cu at (91.3, 57.7)
- added REF**: TestPoint_Pad_1.0x1.0mm, TestPoint:TestPoint_Pad_1.0x1.0mm, B.Cu at (219.6, 99.1)
- added REF**: TestPoint_Pad_1.0x1.0mm, TestPoint:TestPoint_Pad_1.0x1.0mm, B.Cu at (225.8, 114.3)
- added REF**: TestPoint_Pad_1.0x1.0mm, TestPoint:TestPoint_Pad_1.0x1.0mm, B.Cu at (221.5, 114.3)
- added REF**: TestPoint_Pad_1.0x1.0mm, TestPoint:TestPoint_Pad_1.0x1.0mm, B.Cu at (93.7, 78.4)
- added REF**: TestPoint_Pad_1.0x1.0mm, TestPoint:TestPoint_Pad_1.0x1.0mm, B.Cu at (107.2, 121.9)
- added REF**: TestPoint_Pad_1.0x1.0mm, TestPoint:TestPoint_Pad_1.0x1.0mm, B.Cu at (107.2, 126.0)
- added REF**: TestPoint_Pad_1.0x1.0mm, TestPoint:TestPoint_Pad_1.0x1.0mm, B.Cu at (107.1, 102.0)
- added REF**: TestPoint_Pad_1.0x1.0mm, TestPoint:TestPoint_Pad_1.0x1.0mm, B.Cu at (107.1, 104.0)
- added REF**: TestPoint_Pad_1.0x1.0mm, TestPoint:TestPoint_Pad_1.0x1.0mm, B.Cu at (223.6, 114.3)
- added REF**: TestPoint_Pad_1.0x1.0mm, TestPoint:TestPoint_Pad_1.0x1.0mm, B.Cu at (107.2, 124.0)
- added REF**: TestPoint_Pad_1.0x1.0mm, TestPoint:TestPoint_Pad_1.0x1.0mm, F.Cu at (107.2, 126.0)
- added REF**: TestPoint_Pad_1.0x1.0mm, TestPoint:TestPoint_Pad_1.0x1.0mm, F.Cu at (219.3, 114.3)
- added REF**: TestPoint_Pad_1.0x1.0mm, TestPoint:TestPoint_Pad_1.0x1.0mm, F.Cu at (221.5, 114.3)
- added REF**: D_SOD-110, Diode_SMD:D_SOD-110, F.Cu at (107.2, 119.2)
- FPC (x2): moved to B.Cu
- moved REF** 7.43 mm to (62.2, 65.6)
- moved REF** 6.77 mm to (246.7, 65.3)
- moved 33 nF 3.10 mm to (233.8, 121.3), turned to -90 degrees
- moved REF** 0.29 mm to (116.2, 55.0)
- moved REF** 0.29 mm to (106.0, 55.0)
- moved B_Sav 0.25 mm to (96.9, 141.0)
- turned FPC to 90 degrees
- turned FPC to -90 degrees
Routing:
- net (no net): track 1644.5 -> 2133.8 mm, vias 48 -> 68
Other:
- board size 208.7 x 88.9 mm -> 194.7 x 88.9 mm
- board text added: "13"
- board text added: "14"
- board text added: "7"
- board text added: "8"
- board text added: "DSP_PW"
